Commit message: edit hospital scenario people positions and animations, fixed robot not moving when setting goal pose and localization map drift

File: ros2_ws/src/amr_gazebo/urdf/hospital_amr.urdf (robot description, URDF)
Before this commit: robot hospital_amr, 6 links, 5 joints
Joints:
- joint lidar_joint: origin xyz=0 0 0.475 rpy=0 0 0 -> xyz=0 0 0.555 rpy=0 0 0

Commit message: changed size of amr

File: ros2_ws/src/amr_gazebo/urdf/hospital_amr.urdf (robot description, URDF)
Before this commit: robot hospital_amr, 6 links, 5 joints
Links:
- link base_link: geometry collision box size=0.5 0.4 0.3; visual box size=0.8 0.6 0.4
Joints:
- joint camera_joint: origin xyz=0.4 0 0.3 rpy=0 0 0 -> xyz=0.25 0 0.25 rpy=0 0 0
- joint caster_wheel_joint: origin xyz=0.35 0 0.08 rpy=0 0 0 -> xyz=-0.22 0 0.08 rpy=0 0 0
- joint left_wheel_joint: origin xyz=0 0.34 0.15 rpy=0 0 0 -> xyz=0.1 0.22 0.15 rpy=0 0 0
- joint right_wheel_joint: origin xyz=0 -0.34 0.15 rpy=0 0 0 -> xyz=0.1 -0.22 0.15 rpy=0 0 0

Commit message: shrink amr and edit test runner so nav2 does not crash or timeout

File: ros2_ws/src/amr_gazebo/urdf/hospital_amr.urdf (robot description, URDF)
Before this commit: robot hospital_amr, 6 links, 5 joints
Links:
- link base_link: geometry collision box size=0.25 0.2 0.15; visual box size=0.4 0.3 0.2
- link caster_wheel: geometry collision sphere radius=0.04; visual sphere radius=0.04
- link left_wheel: geometry collision cylinder length=0.04 radius=0.075; visual cylinder length=0.04 radius=0.075
- link right_wheel: geometry collision cylinder length=0.04 radius=0.075; visual cylinder length=0.04 radius=0.075
Joints:
- joint camera_joint: origin xyz=0.25 0 0.25 rpy=0 0 0 -> xyz=0.125 0 0.125 rpy=0 0 0
- joint caster_wheel_joint: origin xyz=-0.22 0 0.08 rpy=0 0 0 -> xyz=-0.11 0 0.04 rpy=0 0 0
- joint left_wheel_joint: origin xyz=0.1 0.22 0.15 rpy=0 0 0 -> xyz=0.05 0.11 0.075 rpy=0 0 0
- joint lidar_joint: origin xyz=0 0 0.555 rpy=0 0 0 -> xyz=0 0 0.2775 rpy=0 0 0
- joint right_wheel_joint: origin xyz=0.1 -0.22 0.15 rpy=0 0 0 -> xyz=0.05 -0.11 0.075 rpy=0 0 0

Commit message: add test_runner.py headless mode for faster testing

File: ros2_ws/src/amr_gazebo/urdf/hospital_amr.urdf (robot description, URDF)
Before this commit: robot hospital_amr, 6 links, 5 joints
Links:
- link base_link: geometry collision box size=0.8 0.45 0.4; visual box size=0.8 0.45 0.4
- link camera_link: geometry collision box size=0.12 0.15 0.12; visual box size=0.12 0.15 0.12
- link caster_wheel: geometry collision sphere radius=0.08; visual sphere radius=0.08
- link left_wheel: geometry collision cylinder length=0.08 radius=0.15; visual cylinder length=0.08 radius=0.15
- link right_wheel: geometry collision cylinder length=0.08 radius=0.15; visual cylinder length=0.08 radius=0.15
Joints:
- joint camera_joint: origin xyz=0.125 0 0.125 rpy=0 0 0 -> xyz=0.4 0 0.3 rpy=0 0 0
- joint caster_wheel_joint: origin xyz=-0.11 0 0.04 rpy=0 0 0 -> xyz=0.35 0 0.08 rpy=0 0 0
- joint left_wheel_joint: origin xyz=0.05 0.11 0.075 rpy=0 0 0 -> xyz=0 0.255 0.15 rpy=0 0 0
- joint lidar_joint: origin xyz=0 0 0.2775 rpy=0 0 0 -> xyz=0 0 0.58 rpy=0 0 0
- joint right_wheel_joint: origin xyz=0.05 -0.11 0.075 rpy=0 0 0 -> xyz=0 -0.255 0.15 rpy=0 0 0
